Commit message: thesis update

File: nav2_minimal_tb4_description/urdf/icreate/bumper.urdf.xacro (robot description, xacro)
@@ -24,15 +24,23 @@
   <link name="${link_name}">
     <visual>
+      <origin xyz="0.015 0 0" rpy="0 0 0"/>
       <geometry>
-        <mesh filename="${visual_mesh}"/>
+        <cylinder radius="0.17" length="0.03"/>
       </geometry>
+      <material name="darkgrey">
+        <color rgba="0.2 0.2 0.2 1"/>
+      </material>
     </visual>
     <collision>
+      <origin xyz="0.015 0 0" rpy="0 0 0"/>
       <geometry>
-        <mesh filename="${collision_mesh}"/>
+        <cylinder radius="0.164" length="0.03"/>
       </geometry>
     </collision>
     <xacro:insert_block name="inertial"/>
   </link>
+  <gazebo reference="${link_name}">
+    <material>Gazebo/DarkGrey</material>
+  </gazebo>
   <xacro:dummy_bumper_zone
       name="bump_front_center">

File: nav2_minimal_tb4_description/urdf/icreate/caster.urdf.xacro (robot description, xacro)
@@ -30,8 +30,10 @@
   <gazebo reference="${name}_link">
     <material>Gazebo/DarkGrey</material>
-    <mu1>0.1</mu1>
-    <mu2>0.1</mu2>
-    <kp>1000000.0</kp>
-    <kd>1.0</kd>
+    <mu1>0.0</mu1>
+    <mu2>0.0</mu2>
+    <slip1>0.2</slip1>
+    <slip2>0.2</slip2>
+    <kp>200000.0</kp>
+    <kd>5.0</kd>
   </gazebo>
 </xacro:macro>

File: nav2_minimal_tb4_description/urdf/icreate/create3.urdf.xacro (robot description, xacro)
@@ -12,5 +12,6 @@
   <!-- Mechanical properties -->
   <xacro:property name="body_z_offset"           value="${-2.5*cm2m}" />
-  <xacro:property name="body_collision_z_offset" value="${1*cm2m}" />
+  <!-- Raise collision up to avoid floor penetration when spawning (more clearance) -->
+  <xacro:property name="body_collision_z_offset" value="${3*cm2m}" />
   <xacro:property name="body_mass"               value="2.300" />
   <xacro:property name="body_radius"             value="${16.4*cm2m}" />
@@ -31,11 +32,14 @@
   <link name="base_link">
     <visual>
-      <origin xyz="0 0 ${body_z_offset + base_link_z_offset}" rpy="0 0 ${pi/2}"/>
+      <origin xyz="0 0 ${body_z_offset + base_link_z_offset}" rpy="0 0 0"/>
       <geometry>
-        <mesh filename="package://nav2_minimal_tb4_description/meshes/body_visual.dae" />
+        <cylinder length="${body_length}" radius="${body_radius}"/>
       </geometry>
+      <material name="darkgrey">
+        <color rgba="0.3 0.3 0.3 1"/>
+      </material>
     </visual>
     <collision name="create3_base_collision">
-      <origin xyz="0 0 ${body_z_offset + body_collision_z_offset  + base_link_z_offset}" rpy="0 0 ${pi/2}"/>
+      <origin xyz="0 0 ${body_z_offset + body_collision_z_offset  + base_link_z_offset}" rpy="0 0 0"/>
       <geometry>
         <cylinder length="${body_length}" radius="${body_radius}"/>
@@ -94,7 +98,7 @@
         <max_angular_velocity>2.0</max_angular_velocity>
         <min_angular_velocity>-2.0</min_angular_velocity>
-        <topic>/cmd_vel</topic>
-        <odom_topic>/odom</odom_topic>
-        <tf_topic>tf</tf_topic>
+        <topic>$(arg namespace)/cmd_vel</topic>
+        <odom_topic>$(arg namespace)/odom</odom_topic>
+        <tf_topic>$(arg namespace)/tf</tf_topic>
         <frame_id>odom</frame_id>
         <child_frame_id>base_link</child_frame_id>
@@ -106,5 +110,5 @@
         <joint_name>left_wheel_joint</joint_name>
         <joint_name>right_wheel_joint</joint_name>
-        <topic>joint_states</topic>
+        <topic>$(arg namespace)/joint_states</topic>
         <update_rate>30</update_rate>
       </plugin>

File: nav2_minimal_tb4_description/urdf/icreate/wheel.urdf.xacro (robot description, xacro)
@@ -30,9 +30,11 @@
   </link>
   <gazebo reference="${wheel_link_name}">
-    <mu1>1.0</mu1>
-    <mu2>1.0</mu2>
-    <kp>1000000.0</kp>
-    <kd>100.0</kd>
-    <minDepth>0.0001</minDepth>
+    <mu1>0.9</mu1>
+    <mu2>0.9</mu2>
+    <slip1>0.1</slip1>
+    <slip2>0.1</slip2>
+    <kp>200000.0</kp>
+    <kd>20.0</kd>
+    <minDepth>0.001</minDepth>
     <maxVel>1.0</maxVel>
     <material>Gazebo/DarkGrey</material>

File: nav2_minimal_tb4_description/urdf/sensors/camera_bracket.urdf.xacro (robot description, xacro)
@@ -13,8 +13,18 @@
   <link name="${link_name}">
     <visual>
+      <origin xyz="-0.01 0 0" rpy="0 0 0"/>
       <geometry>
-       <mesh filename="package://nav2_minimal_tb4_description/meshes/camera_bracket.dae" scale="1 1 1" />
+        <box size="0.04 0.14 0.06"/>
       </geometry>
+      <material name="darkgrey">
+        <color rgba="0.1 0.1 0.1 1"/>
+      </material>
     </visual>
+    <collision>
+      <origin xyz="-0.01 0 0" rpy="0 0 0"/>
+      <geometry>
+        <box size="0.04 0.14 0.06"/>
+      </geometry>
+    </collision>
     <inertial>
       <mass value="${mass}"/>
@@ -23,4 +33,7 @@
     </inertial>
   </link>
+  <gazebo reference="${link_name}">
+    <material>Gazebo/DarkGrey</material>
+  </gazebo>
   <gazebo reference="${joint_name}">
     <preserveFixedJoint>true</preserveFixedJoint>

File: nav2_minimal_tb4_description/urdf/sensors/oakd.urdf.xacro (robot description, xacro)
@@ -1,5 +1,5 @@
 <?xml version="1.0"?>
 <robot xmlns:xacro="http://ros.org/wiki/xacro">
-<xacro:macro name="oakd" params="name:=oakd parent_link *origin model:=pro">
+<xacro:macro name="oakd" params="name:=oakd parent_link *origin model:=pro namespace:=''">
   <xacro:include filename="$(find nav2_minimal_tb4_description)/urdf/icreate/common_properties.urdf.xacro"/>
   <xacro:property name="mass"       value="0.061"/>
@@ -21,7 +21,11 @@
   <link name="${base_frame}">
     <visual>
+      <origin xyz="${collision_offset_x} ${collision_offset_y} ${collision_offset_z}" rpy="0 0 0"/>
       <geometry>
-        <mesh filename="package://nav2_minimal_tb4_description/meshes/${name}_${model}.dae" scale="1 1 1" />
+        <box size="${collision_length_x} ${collision_length_y} ${collision_length_z}"/>
       </geometry>
+      <material name="darkgrey">
+        <color rgba="0.15 0.15 0.15 1"/>
+      </material>
     </visual>
     <collision>
@@ -37,4 +41,7 @@
     </inertial>
   </link>
+  <gazebo reference="${base_frame}">
+    <material>Gazebo/DarkGrey</material>
+  </gazebo>
   <!-- RGB Camera -->
   <link name="${name}_rgb_camera_frame">
@@ -114,6 +121,6 @@
       </camera>
       <update_rate>10</update_rate>
-      <visualize>true</visualize>
-      <topic>rgbd_camera</topic>
+      <visualize>false</visualize>
+      <topic>${namespace}/rgbd_camera</topic>
     </sensor>
     <xacro:material_darkgray/>

File: nav2_minimal_tb4_description/urdf/sensors/rplidar.urdf.xacro (robot description, xacro)
@@ -1,5 +1,5 @@
 <?xml version="1.0"?>
 <robot xmlns:xacro="http://ros.org/wiki/xacro">
-<xacro:macro name="rplidar" params="name parent_link gazebo *origin">
+<xacro:macro name="rplidar" params="name parent_link gazebo namespace:='' *origin">
   <xacro:include filename="$(find nav2_minimal_tb4_description)/urdf/icreate/common_properties.urdf.xacro"/>
   <xacro:property name="mass"       value="0.17"/>
@@ -31,7 +31,7 @@
   <gazebo reference="${name}_link">
     <xacro:ray_sensor sensor_name="${name}" gazebo="${gazebo}"
-                  update_rate="10.0" visualize="true"
+                  update_rate="10.0" visualize="false"
                   h_samples="360" h_res="1.0" h_min_angle="0.000" h_max_angle="6.280000"
-                  r_min="0.164" r_max="20.0" r_res="0.01">
+                  r_min="0.164" r_max="20.0" r_res="0.01" namespace="${namespace}">
                   <plugin name="dummy" filename="dummyfile"></plugin>
     </xacro:ray_sensor>

File: nav2_minimal_tb4_description/urdf/standard/tower_sensor_plate.urdf.xacro (robot description, xacro)
@@ -13,7 +13,11 @@
   <link name="${link_name}">
     <visual>
+      <origin xyz="0 0 0.001" rpy="0 0 0"/>
       <geometry>
-       <mesh filename="package://nav2_minimal_tb4_description/meshes/tower_sensor_plate.dae" scale="1 1 1" />
+        <cylinder radius="0.137" length="0.003"/>
       </geometry>
+      <material name="darkgrey">
+        <color rgba="0.1 0.1 0.1 1"/>
+      </material>
     </visual>
     <collision>
@@ -29,4 +33,7 @@
     </inertial>
   </link>
+  <gazebo reference="${link_name}">
+    <material>Gazebo/DarkGrey</material>
+  </gazebo>
   <gazebo reference="${joint_name}">
     <preserveFixedJoint>true</preserveFixedJoint>

File: nav2_minimal_tb4_description/urdf/standard/tower_standoff.urdf.xacro (robot description, xacro)
@@ -13,8 +13,11 @@
   <link name="${link_name}">
     <visual>
-      <origin rpy="0 ${pi/2} 0"/>
+      <origin xyz="0 0 0" rpy="0 0 0"/>
       <geometry>
-       <mesh filename="package://nav2_minimal_tb4_description/meshes/tower_standoff.dae" scale="1 1 1" />
+        <cylinder radius="0.006" length="0.205"/>
       </geometry>
+      <material name="darkgrey">
+        <color rgba="0.1 0.1 0.1 1"/>
+      </material>
     </visual>
     <collision>
@@ -30,4 +33,7 @@
     </inertial>
   </link>
+  <gazebo reference="${link_name}">
+    <material>Gazebo/DarkGrey</material>
+  </gazebo>
   <gazebo reference="${joint_name}">
     <preserveFixedJoint>true</preserveFixedJoint>

File: nav2_minimal_tb4_description/urdf/standard/turtlebot4.urdf.xacro (robot description, xacro)
@@ -1,8 +1,13 @@
 <?xml version="1.0" ?>
 <robot name="turtlebot4" xmlns:xacro="http://ros.org/wiki/xacro">
+  <!-- Namespace for Gazebo topics -->
+  <xacro:arg name="namespace" default=""/>
+  <!-- Enable/disable RPLIDAR sensor (set to 0 to disable for performance testing) -->
+  <xacro:property name="enable_rplidar" value="0" />
   <!-- Base create3 model -->
   <xacro:include filename="$(find nav2_minimal_tb4_description)/urdf/icreate/create3.urdf.xacro" />
   <xacro:include filename="$(find nav2_minimal_tb4_description)/urdf/sensors/rplidar.urdf.xacro" />
   <xacro:include filename="$(find nav2_minimal_tb4_description)/urdf/sensors/oakd.urdf.xacro" />
+  <xacro:include filename="$(find nav2_minimal_tb4_description)/urdf/sensors/proximity.urdf.xacro" />
   <xacro:include filename="$(find nav2_minimal_tb4_description)/urdf/sensors/camera_bracket.urdf.xacro" />
   <xacro:include filename="$(find nav2_minimal_tb4_description)/urdf/standard/tower_standoff.urdf.xacro" />
@@ -60,12 +65,16 @@
   <link name="shell_link">
     <visual>
-      <origin xyz="0 0 0" rpy="${pi/2} 0 ${pi/2}"/>
+      <origin xyz="0 0 0" rpy="0 0 0"/>
       <geometry>
-        <mesh filename="package://nav2_minimal_tb4_description/meshes/shell.dae" scale="1 1 1" />
+        <box size="${shell_length} ${shell_radius*2} 0.08"/>
       </geometry>
+      <material name="darkgrey">
+        <color rgba="0.2 0.2 0.2 1"/>
+      </material>
     </visual>
     <collision name="shell_collision">
+      <origin xyz="0 0 0" rpy="0 0 0"/>
       <geometry>
-        <mesh filename="package://nav2_minimal_tb4_description/meshes/shell_collision.dae" scale="1 1 1" />
+        <box size="${shell_length} ${shell_radius*2} 0.08"/>
       </geometry>
     </collision>
@@ -110,13 +119,29 @@
   </xacro:tower_sensor_plate>
   <!-- Turtlebot4 sensor definitions -->
-  <xacro:rplidar name="rplidar" parent_link="shell_link" gazebo="$(arg gazebo)">
-    <origin xyz="${rplidar_x_offset} ${rplidar_y_offset} ${rplidar_z_offset}"
-            rpy="0 0 ${pi/2}"/>
-  </xacro:rplidar>
+  <xacro:if value="${enable_rplidar}">
+    <xacro:rplidar name="rplidar" parent_link="shell_link" gazebo="$(arg gazebo)" namespace="$(arg namespace)">
+      <origin xyz="${rplidar_x_offset} ${rplidar_y_offset} ${rplidar_z_offset}"
+              rpy="0 0 ${pi/2}"/>
+    </xacro:rplidar>
+  </xacro:if>
   <xacro:camera_bracket name="oakd_camera_bracket">
     <origin xyz="${camera_mount_x_offset} ${camera_mount_y_offset} ${camera_mount_z_offset}"/>
   </xacro:camera_bracket>
-  <xacro:oakd model="pro" parent_link="oakd_camera_bracket">
+  <xacro:oakd model="pro" parent_link="oakd_camera_bracket" namespace="$(arg namespace)">
     <origin xyz="${oakd_pro_x_offset} ${oakd_pro_y_offset} ${oakd_pro_z_offset}"/>
   </xacro:oakd>
+  <!-- Proximity sensors ring on base_link -->
+  <xacro:proximity_ring parent_link="base_link" gazebo="$(arg gazebo)" namespace="$(arg namespace)" radius="0.16" z_offset="0.05"/>
+  <!-- Ground truth odometry publisher for Gazebo -->
+  <xacro:arg name="gazebo" default=""/>
+  <xacro:if value="${('$(arg gazebo)' == 'ignition' or '$(arg gazebo)' == 'gazebo')}">
+    <gazebo>
+      <plugin filename="libgz-sim-odometry-publisher-system.so" name="gz::sim::systems::OdometryPublisher">
+        <odom_topic>$(arg namespace)/ground_truth_odom</odom_topic>
+        <odom_frame>mission</odom_frame>
+        <robot_base_frame>base_footprint</robot_base_frame>
+        <odom_publish_frequency>10</odom_publish_frequency>
+      </plugin>
+    </gazebo>
+  </xacro:if>
 </robot>

File: nav2_minimal_tb4_description/urdf/standard/weight_block.urdf.xacro (robot description, xacro)
@@ -13,8 +13,18 @@
   <link name="${link_name}">
     <visual>
+      <origin xyz="0.05 0 0" rpy="0 0 0"/>
       <geometry>
-       <mesh filename="package://nav2_minimal_tb4_description/meshes/weight_block.dae" scale="1 1 1" />
+        <box size="0.10 0.035 0.035"/>
       </geometry>
+      <material name="darkgrey">
+        <color rgba="0.15 0.15 0.15 1"/>
+      </material>
     </visual>
+    <collision>
+      <origin xyz="0.05 0 0" rpy="0 0 0"/>
+      <geometry>
+        <box size="0.10 0.035 0.035"/>
+      </geometry>
+    </collision>
     <inertial>
       <origin xyz="0.1 0 0"/>
@@ -24,4 +34,7 @@
     </inertial>
   </link>
+  <gazebo reference="${link_name}">
+    <material>Gazebo/DarkGrey</material>
+  </gazebo>
   <gazebo reference="${joint_name}">
     <preserveFixedJoint>true</preserveFixedJoint>
